Commit message: added first plate

File: spike_description/urdf/spike.urdf.xacro (robot description, xacro)
@@ -7,4 +7,29 @@
 -->
 <robot name="spike" xmlns:xacro="http://ros.org/wiki/xacro">
-  <xacro:include filename="$(find roomba_description)/urdf/white_roomba.urdf.xacro" />
+	<xacro:include filename="$(find roomba_description)/urdf/white_roomba.urdf.xacro" />
+        <!-- base link, basically the body of the Roomba -->
+        <link name="first_plate">
+                <inertial>
+                        <mass value="2" />
+                        <origin xyz="0 0 0.0" />
+                        <inertia ixx="0.01" ixy="0.0" ixz="0.0" iyy="0.01" iyz="0.0" izz="0.5" />
+                </inertial>
+                <visual>
+                        <origin xyz=" 0 0 0.0308" rpy="0 0 1.5708" />
+                        <geometry>
+                                <cylinder length="0.0032" radius="0.1524"/>
+                        </geometry>
+                </visual>
+                <collision>
+                        <origin xyz="0.0 0.0 0.0308" rpy="0 0 0" />
+                        <geometry>
+                                <cylinder length="0.0032" radius="0.1524"/>
+                        </geometry>
+                </collision>
+        </link>
+	<joint name="base_to_first_plate" type="fixed">
+		<parent link="base_link"/>
+		<child link="first_plate"/>
+                <origin xyz="0.0 0.0 0.0816" rpy="0 0 0" />
+	</joint>
 </robot>

Commit message: made plates white.  added 2nd plate.  imported xtion model from iheartengineering's turtlebot description.

File: spike_description/urdf/spike.urdf.xacro (robot description, xacro)
@@ -7,6 +7,8 @@
 -->
 <robot name="spike" xmlns:xacro="http://ros.org/wiki/xacro">
-	<xacro:include filename="$(find roomba_description)/urdf/white_roomba.urdf.xacro" />
-        <!-- base link, basically the body of the Roomba -->
+        <material name="White">
+                <color rgba="1 1 1 1"/>
+        </material>
+	<xacro:include filename="$(find roomba_description)/urdf/roomba.urdf.xacro" />
         <link name="first_plate">
                 <inertial>
@@ -20,4 +22,5 @@
                                 <cylinder length="0.0032" radius="0.1524"/>
                         </geometry>
+		        <material name="White"/>
                 </visual>
                 <collision>
@@ -33,3 +36,30 @@
                 <origin xyz="0.0 0.0 0.0816" rpy="0 0 0" />
 	</joint>
+        <link name="top_plate">
+                <inertial>
+                        <mass value="2" />
+                        <origin xyz="0 0 0.0" />
+                        <inertia ixx="0.01" ixy="0.0" ixz="0.0" iyy="0.01" iyz="0.0" izz="0.5" />
+                </inertial>
+                <visual>
+                        <origin xyz=" 0 0 0.0" rpy="0 0 1.5708" />
+                        <geometry>
+                                <box size=".1 .1 .001"/>
+                        </geometry>
+		        <material name="White"/>
+                </visual>
+                <collision>
+                        <origin xyz="0.0 0.0 0.0" rpy="0 0 0" />
+                        <geometry>
+                                <box size=".1 .1 .001"/>
+                        </geometry>
+                </collision>
+        </link>
+	<joint name="first_plate_to_top_plate" type="fixed">
+		<parent link="first_plate"/>
+		<child link="top_plate"/>
+                <origin xyz="-0.1 0.0 0.1016" rpy="0 0 0" />
+	</joint>
+        <xacro:include filename="$(find turtlebot_xtion_top_description)/urdf/xtion.xacro" />
+   	<xacro:xtion parent="top_plate" x_loc="0" y_loc="0" z_loc="0" rr="0" rp="0" ry="0"/>
 </robot>

Commit message: Added imu_link to urdf

File: spike_description/urdf/spike.urdf.xacro (robot description, xacro)
@@ -10,4 +10,7 @@
                 <color rgba="1 1 1 1"/>
         </material>
+       <material name="Blue">
+                <color rgba="0 0.75 1 1"/>
+        </material>
 	<xacro:include filename="$(find roomba_description)/urdf/roomba.urdf.xacro" />
         <link name="first_plate">
@@ -18,5 +21,5 @@
                 </inertial>
                 <visual>
-                        <origin xyz=" 0 0 0.0308" rpy="0 0 1.5708" />
+                        <origin xyz=" 0 0 0" rpy="0 0 1.5708" />
                         <geometry>
                                 <cylinder length="0.0032" radius="0.1524"/>
@@ -25,5 +28,5 @@
                 </visual>
                 <collision>
-                        <origin xyz="0.0 0.0 0.0308" rpy="0 0 0" />
+                        <origin xyz="0.0 0.0 0" rpy="0 0 0" />
                         <geometry>
                                 <cylinder length="0.0032" radius="0.1524"/>
@@ -34,6 +37,19 @@
 		<parent link="base_link"/>
 		<child link="first_plate"/>
-                <origin xyz="0.0 0.0 0.0816" rpy="0 0 0" />
+                <origin xyz="0.0 0.0 0.1124" rpy="0 0 0" />
 	</joint>
+        <link name="imu_link">
+                <visual>
+                        <geometry>
+                                <box size=".0159 .0206 .0033"/>
+                        </geometry>
+		                <material name="Blue"/>
+                </visual>
+        </link>
+    	<joint name="first_plate_to_imu" type="fixed">
+			<parent link="first_plate"/>
+			<child link="imu_link"/>
+            <origin xyz="0 0 0.003" rpy="0 0 0" />
+        </joint>
         <link name="top_plate">
                 <inertial>
